File: pcb/purify_io.kicad_sch (KiCad schematic)
At the start: 0 parts

Commit message: WIP power regulation for PCB
Parts:
- added C1, C3: 1uF, Capacitor_SMD:C_0603_1608Metric, symbol Device:C_Small
- added C2, C4: 10pF, Capacitor_SMD:C_0603_1608Metric, symbol Device:C_Small
- added C2, C4: 10uF, Capacitor_SMD:C_0603_1608Metric, symbol Device:C_Small
- added C5, C6 (x2), C7, C8: 100nF, Capacitor_SMD:C_0603_1608Metric, symbol Device:C_Small
- added C7: 4u7F, Capacitor_SMD:C_0603_1608Metric, symbol Device:C_Small
- added FB1: 120R, Inductor_SMD:L_0603_1608Metric, symbol Device:FerriteBead_Small
- added J2: Programmer Conn, Connector:Tag-Connect_TC2030-IDC-FP_2x03_P1.27mm_Vertical, symbol ATL:TC2030
- added R5: 10k, Resistor_SMD:R_0603_1608Metric, symbol Device:R_Small_US
- added U1: STM32F411CCUx, Package_DFN_QFN:QFN-48-1EP_7x7mm_P0.5mm_EP5.6x5.6mm, symbol MCU_ST_STM32F4:STM32F411CCUx
- added Y1: 16MHz, Crystal:Crystal_SMD_Abracon_ABM8G-4Pin_3.2x2.5mm, symbol Device:Crystal_GND24_Small
Connections:
- new net: C2.1, U1.5 (PH0), Y1.1
- new net: C4.1, U1.6 (PH1), Y1.3
- new net: C7.2, U1.22 (VCAP1)
- new net: J2.3 (~{RESET}), R5.2
- new net +3.3V: C1.1, C4.1, C5.1, C6.1, C7.1, C8.1, FB1.1, U1.1 (VBAT), U1.24 (VDD), U1.36 (VDD), U1.48 (VDD)
- new net +3.3VA: C2.1, C3.1, FB1.2, U1.9 (VDDA)
- new net GND: C1.2, C2.2, C2.2, C3.2, C4.2, C4.2, C5.2, C6.1, C6.2, C7.1, C7.2, C8.2, J2.5 (GND), U1.23 (VSS), U1.35 (VSS), U1.47 (VSS), U1.49 (VSS), U1.8 (VSSA), Y1.2, Y1.4
- new net SWCLK: J2.4 (SWCLK)
- new net SWDIO: J2.2 (SWDIO)
- new net SWO: J2.6 (SWO)
- new net ~{RESET}: C6.2, R5.1, U1.7 (NRST)
- no-connect marks 0 -> 1
Other:
- added sheet Power Regulator (power_regulator.kicad_sch)
